File: 8-channel/smartcitizen-adc-8ch.kicad_pcb (KiCad board)
At the start: 2 copper layers, 46.9 x 46.9 mm, 34 parts, among them J1 GROVE1, J2 GROVE2, J3 EXT_V, J4 EXT_V, J5 Conn_02x05_Odd_Even, M1 PINHD-1x06-HEADER, M2 PINHD-1x06-HEADER, M3 PINHD-1x06-HEADER, M4 PINHD-1x06-HEADER, M5 PINHD-1x02-HEADER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

Commit message: 8-channel footprint
Other:
- board text added: "SmartCitizen ASB 8-ch I2C I2C-V: 3.3V to EXT-V EXT-V: I2C-V to 5.5V"
- board text removed: "SmartCitizen ASB 8-ch I2C-V: 3.3V to EXT-V EXT-V: I2C-V to 5.5V"
Changed lines of the file:
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@@
       (outputformat 1)
       (mirror false)
-      (drillshape 1)
+      (drillshape 0)
       (scaleselection 1)
-      (outputdirectory ""))
+      (outputdirectory "exports/"))
   )
   (net 0 "")
@@
     (effects (font (size 0.8 0.8) (thickness 0.12)))
   )
-  (gr_text "SmartCitizen ASB\n8-ch\nI2C-V: 3.3V to EXT-V\nEXT-V: I2C-V to 5.5V" (at 157.0863 95.41764) (layer B.SilkS)
+  (gr_text "SmartCitizen ASB\n8-ch I2C\nI2C-V: 3.3V to EXT-V\nEXT-V: I2C-V to 5.5V" (at 157.0863 95.41764) (layer B.SilkS)
     (effects (font (size 1 1) (thickness 0.15)) (justify left mirror))
   )
