File: 8-channel/smartcitizen-adc-8ch-step.sch (KiCad schematic (older format))
At the start: 46 parts, among them J1 GROVE1, J2 GROVE2, J5 Conn_02x05_Odd_Even, M1 PINHD-1x06-HEADER, M2 PINHD-1x06-HEADER, M3 PINHD-1x06-HEADER, M4 PINHD-1x06-HEADER, T1 NMOSFETSOT23, T2 NMOSFETSOT23, U1 ADS1115IDGSR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

Commit message: Update to new 8-channel board
Parts:
- C12, C3, C8: footprint fab-C1206FAB -> Capacitor_SMD:C_0805_2012Metric_Pad1.18x1.45mm_HandSolder; LCSC C1944 -> C107135; MFR.Part # CL31B103KGFNNNE -> CC0805KRX7R0BB103; Manufacturer Samsung Electro-Mechanics -> YAGEO
- C13, C4, C9: footprint fab-C1206FAB -> Capacitor_SMD:C_0805_2012Metric_Pad1.18x1.45mm_HandSolder; LCSC C24497 -> C111492; MFR.Part # CL31B104KBCNNNC -> CC0805JRX7R9BB104; Manufacturer Samsung Electro-Mechanics -> YAGEO
- M1, M2, M3, M4: footprint Connector_PinHeader_2.54mm:PinHeader_1x06_P2.54mm_Vertical -> Connector_Molex:Molex_KK-254_AE-6410-06A_1x06_P2.54mm_Vertical
Other:
- note added: "Notes:\nMOLEX 6x1 2.54mm Male: 22232061\nTOBY 1.28"
- note removed: "Notes:\nMOLEX 6x1 2.54mm Male: 22232061\nTOBY 1.28\nScrew Connector: Phoenix Contact 1985807 (same as PS)\nUSB A - Phoenix Contact 87520-1110BLF\nMASTER POWER CUT - Vishay SiP32431 SC-70\n"

Commit message: 8-channel board changes and schematic
Parts:
- C10: value 100nF -> 330nF; LCSC C24497 -> C307572; MFR.Part # CL31B104KBCNNNC -> CL31B334KBFNNNE
- R10, R11: footprint Resistor_SMD:R_01005_0402Metric -> Resistor_SMD:R_0402_1005Metric
- U5: value LM3480-5.0 -> PJ78605SA; LCSC C128407 -> C411751
Changed lines of the file:
@@
 F 0 "R10" H 9700 2000 45  0000 L CNN
 F 1 "1kΩ" H 9650 1800 45  0000 L CNN
-F 2 "Resistor_SMD:R_01005_0402Metric" H 9780 2050 20  0001 C CNN
+F 2 "Resistor_SMD:R_0402_1005Metric" H 9780 2050 20  0001 C CNN
 F 3 "https://datasheet.lcsc.com/szlcsc/Uniroyal-Elec-0402WGF1001TCE_C11702.pdf" H 9750 1900 50  0001 C CNN
 F 4 "Uniroyal Elec" H 9750 1900 50  0001 C CNN "Manufacturer"
@@
 F 0 "R11" H 9700 1600 45  0000 L CNN
 F 1 "1kΩ" H 9650 1400 45  0000 L CNN
-F 2 "Resistor_SMD:R_01005_0402Metric" H 9780 1650 20  0001 C CNN
+F 2 "Resistor_SMD:R_0402_1005Metric" H 9780 1650 20  0001 C CNN
 F 3 "https://datasheet.lcsc.com/szlcsc/Uniroyal-Elec-0402WGF1001TCE_C11702.pdf" H 9750 1500 50  0001 C CNN
 F 4 "Uniroyal Elec" H 9750 1500 50  0001 C CNN "Manufacturer"
@@
 P 9900 4150
 F 0 "U5" H 9900 4392 50  0000 C CNN
-F 1 "LM3480-5.0" H 9900 4301 50  0000 C CNN
+F 1 "PJ78605SA" H 9900 4301 50  0000 C CNN
 F 2 "Package_TO_SOT_SMD:SOT-23" H 9900 4375 50  0001 C CIN
-F 3 "http://www.ti.com/lit/ds/symlink/lm3480.pdf" H 9900 4150 50  0001 C CNN
-F 4 "C128407" H 9900 4150 50  0001 C CNN "LCSC"
+F 3 "https://datasheet.lcsc.com/lcsc/1912111437_PJSEMI-PJ78L05SA_C411751.pdf" H 9900 4150 50  0001 C CNN
+F 4 "C411751" H 9900 4150 50  0001 C CNN "LCSC"
 	1    9900 4150
 	1    0    0    -1
@@
 P 9500 4450
 F 0 "C10" V 9400 4250 45  0000 L CNN
-F 1 "100nF" V 9500 4150 45  0000 L CNN
+F 1 "330nF" V 9500 4150 45  0000 L CNN
 F 2 "fab-C1206FAB" H 9530 4600 20  0001 C CNN
 F 3 "https://datasheet.lcsc.com/szlcsc/Samsung-Electro-Mechanics-CL31B104KBCNNNC_C24497.pdf" H 9500 4450 50  0001 C CNN
 F 4 "Samsung Electro-Mechanics" V 9500 4450 50  0001 C CNN "Manufacturer"
-F 5 "CL31B104KBCNNNC" V 9500 4450 50  0001 C CNN "MFR.Part #"
-F 6 "C24497" V 9500 4450 50  0001 C CNN "LCSC"
+F 5 "CL31B334KBFNNNE" V 9500 4450 50  0001 C CNN "MFR.Part #"
+F 6 "C307572" V 9500 4450 50  0001 C CNN "LCSC"
 	1    9500 4450
 	0    1    1    0
