File: 8-channel-step/smartcitizen-adc-8ch-step.sch (KiCad schematic (older format))
At the start: 51 parts, among them J1 GROVE1, J2 GROVE2, J4 USB_BULGIN, J5 Conn_02x05_Odd_Even, J6 USB_B_Micro, J7 USB_A, M1 PINHD-1x06-HEADER, M2 PINHD-1x06-HEADER, M3 PINHD-1x06-HEADER, M4 PINHD-1x06-HEADER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

Commit message: Stable version fixing address issue
Parts:
- removed C6: 1uF, Capacitor_SMD:C_0805_2012Metric, symbol fab:CAP-UNPOLARIZEDFAB
- removed C7: 100nF, fab-C1206FAB, symbol fab:CAP-UNPOLARIZEDFAB
- removed D1: RED_LED, LED_SMD:LED_0402_1005Metric, symbol Device:LED
- removed J4: USB_BULGIN, Connector_PinHeader_2.54mm:PinHeader_1x05_P2.54mm_Vertical, symbol Connector:Conn_01x05_Female
- removed J6: USB_B_Micro, Connector_USB:USB_Micro-B_XKB-U254-051T-4BH83-F1S_Horizontal, symbol Connector:USB_B_Micro
- removed J7: USB_A, Connector_USB:USB_A_Amphenol_87520-1110BLF, symbol Connector:USB_A
- removed JP1: J3_Bridged12, Jumper:SolderJumper-3_P1.3mm_Bridged12_RoundedPad1.0x1.5mm, symbol Jumper:SolderJumper_3_Bridged12
- removed JP2: Jumper_2_Open, Jumper:SolderJumper-2_P1.3mm_Open_RoundedPad1.0x1.5mm, symbol Jumper:Jumper_2_Open
- removed R9: 1kΩ, Resistor_SMD:R_01005_0402Metric, symbol fab:RES-US1206FAB
- removed U3: SiP32431DR3, Package_TO_SOT_SMD:SOT-363_SC-70-6, symbol Power_Management:SiP32431DR3
- added H1, H2, H3: MountingHole, MountingHole:MountingHole_3.2mm_M3, symbol Mechanical:MountingHole
- added JP2: J3_Bridged12, Jumper:SolderJumper-3_P1.3mm_Bridged12_RoundedPad1.0x1.5mm, symbol Jumper:SolderJumper_3_Bridged12
- added OSH1: Logo_Open_Hardware_Small, Symbol:OSHW-Symbol_6.7x6mm_SilkScreen, symbol Graphic:Logo_Open_Hardware_Small
- FB1, FB2: footprint Resistor_SMD:R_0805_2012Metric -> Resistor_SMD:R_0805_2012Metric_Pad1.20x1.40mm_HandSolder
Connections:
- net labels removed: 5VSEL, D+, D-, VCC_PRE, VUSB
- wire segments 238 -> 195
- no-connect marks 1 -> 0
Other:
- note added: "LED INDICATORS"
- note removed: "GROVE/USB LED INDICATORS"
- note removed: "POWER/USB DATA IN\nUSE EITHER, BUT NOT BOTH"
- moved on the sheet: C12, C13, C3, C4, C8, C9, D2, D3, FB1, FB2, JP4, R1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
